Commit message: experiment: two robots in one urdf_xacro

File: urdf/robot_arm.xacro (robot description, xacro)
@@ -9,9 +9,15 @@
     <xacro:property name="joint_name_4" value="${robot_prefix}joint4" />
     <xacro:property name="joint_name_5" value="${robot_prefix}joint5" />
-  <joint name="${joint_name_1}" type="prismatic">
+    <xacro:property name="link_name_1" value="${robot_prefix}forearm" />
+    <xacro:property name="link_name_2" value="${robot_prefix}uperarm" />
+    <xacro:property name="link_name_3" value="${robot_prefix}gripper" />
+    <xacro:property name="link_name_4" value="${robot_prefix}grippercenter" />
+    <xacro:property name="link_name_5" value="${robot_prefix}base" />
+    <xacro:property name="link_name_6" value="${robot_prefix}pillar" />
+    <joint name="${joint_name_1}" type="prismatic">
       <origin xyz="0.049999999999999975 -0.15 0.050000000000000114" rpy="1.5896965726302545e-17 -2.606945736351794e-17 -1.5707963267948966"/>
       <axis xyz="1 0 0"/>
-      <parent link="test__upperarm"/>
-      <child link="forearm"/>
+      <parent link="${link_name_2}"/>
+      <child link="${link_name_1}"/>
       <limit effort="1000" lower="-1.548" upper="1.548" velocity="0.5"/>
     </joint>
@@ -19,6 +25,6 @@
       <origin xyz="0.5150000099092719 0.0499999999999995 0.025000000000000456" rpy="9.373400549266757e-16 -3.404356883972169e-17 -1.570796326794856"/>
       <axis xyz="1 0 0"/>
-      <parent link="forearm"/>
-      <child link="gripper"/>
+      <parent link="${link_name_1}"/>
+      <child link="${link_name_3}"/>
       <limit effort="1000" lower="-1.548" upper="1.548" velocity="0.5"/>
     </joint>
@@ -26,6 +32,6 @@
       <origin xyz="0.5350000099092719 -9.947598300641403e-17 4.547473508864641e-16" rpy="1.8648277366750716e-16 1.5707963267948961 0.0"/>
       <axis xyz="1 0 0"/>
-      <parent link="forearm"/>
-      <child link="grippercenter"/>
+      <parent link="${link_name_1}"/>
+      <child link="${link_name_3}center"/>
       <limit effort="1000" lower="-1.548" upper="1.548" velocity="0.5"/>
     </joint>
@@ -33,6 +39,6 @@
       <origin xyz="1.130678486794346e-16 -3.551106571559647e-17 0.1" rpy="0.07862783327530606 -1.570796326794895 -0.07862783327530617"/>
       <axis xyz="1 0 0"/>
-      <parent link="base"/>
-      <child link="pillar"/>
+      <parent link="${link_name_5}"/>
+      <child link="${link_name_6}"/>
       <limit effort="1000" lower="-1.548" upper="1.548" velocity="0.5"/>
     </joint>
@@ -40,9 +46,9 @@
       <origin xyz="0.775 1.5706654524051988e-16 1.4001861794794053e-15" rpy="1.570796326794896 -1.1102230246251565e-16 1.5707963267948968"/>
       <axis xyz="1 0 0"/>
-      <parent link="pillar"/>
-      <child link="test__upperarm"/>
+      <parent link="${link_name_6}"/>
+      <child link="${link_name_2}"/>
       <limit effort="1000" lower="-1.548" upper="1.548" velocity="0.5"/>
     </joint>
-    <link name="forearm">
+    <link name="${link_name_1}">
       <visual>
         <origin xyz="-0.1499999999999993 -0.05 -0.9250000000000002" rpy="-3.404356883968544e-17 -8.326057456882182e-16 -1.86482773667507e-16"/>
@@ -55,5 +61,5 @@
       </visual>
     </link>
-    <link name="test__upperarm">
+    <link name="${link_name_2}">
       <visual>
         <origin xyz="-4.252363031521377e-17 -7.478248673434915e-16 -0.875" rpy="-1.814660311338287e-17 -8.586752030517361e-16 -1.5707963267948966"/>
@@ -66,5 +72,5 @@
       </visual>
     </link>
-    <link name="gripper">
+    <link name="${link_name_3}">
       <visual>
         <origin xyz="0.09999999999997242 -0.6650000099092762 -0.9499999999999998" rpy="-2.1385526102475867e-30 1.0473430923845879e-16 1.5707963267948557"/>
@@ -77,6 +83,6 @@
       </visual>
     </link>
-    <link name="grippercenter"/>
-    <link name="base">
+    <link name="${link_name_4}"/>
+    <link name="${link_name_5}">
       <visual>
         <origin xyz="-0.0 -0.0 -0.0" rpy="0.0 -0.0 0.0"/>
@@ -89,5 +95,5 @@
       </visual>
     </link>
-    <link name="pillar">
+    <link name="${link_name_6}">
       <visual>
         <origin xyz="-0.1 2.3264597724122947e-17 -5.3465605014339346e-17" rpy="0.0612461921254255 1.570796326794895 0.06124619212542564"/>
@@ -101,4 +107,4 @@
     </link>
   </xacro:macro>
-  <xacro:my_robot robot_name="test234" />
+  <xacro:my_robot robot_name="${this_robot_name}" />
 </robot>

File: urdf/robotic_cell.urdf.xacro (robot description, xacro)
@@ -1,6 +1,15 @@
 <?xml version="1.0"?>
 <robot xmlns:xacro="http://www.ros.org/wiki/xacro"  name="robotic_cell">
+  <joint name="togehter" type="fixed">
+      <origin xyz="0 1.0 0" rpy="0 0 0"/>
+      <axis xyz="1 0 0"/>
+      <parent link="cell_element1_base"/>
+      <child link="cell_element2_base"/>
+   </joint>
+ <xacro:property name="this_robot_name" value="cell_element1_" />
   <xacro:include filename="$(find robotic_cell_description)/urdf/robot_arm.xacro" >
-    <xacro:arg name="this_robot_name" value="robot_test1" />
+  </xacro:include>
+   <xacro:property name="this_robot_name" value="cell_element2_" />
+  <xacro:include filename="$(find robotic_cell_description)/urdf/robot_arm.xacro" >
   </xacro:include>
 </robot>
