Commit message: experiment: get and use yaml data in xacro

File: urdf/robotic_cell.urdf.xacro (robot description, xacro)
@@ -1,14 +1,18 @@
 <?xml version="1.0"?>
 <robot xmlns:xacro="http://www.ros.org/wiki/xacro"  name="robotic_cell">
+  <xacro:property name="yaml_file" value="$(find robotic_cell_description)/config/active_config.yaml" />
+  <xacro:property name="active_config" value="${load_yaml(yaml_file)}"/>
+  <xacro:property name="current_connection_name" value="first_connection"/>
+  <xacro:property name="connection_config" value="${active_config[current_connection_name]}"/>
   <joint name="togehter" type="fixed">
-      <origin xyz="0 1.0 0" rpy="0 0 0"/>
+      <origin xyz="${connection_config['x']} ${connection_config['y']} ${connection_config['z']}" rpy="0 0 0"/>
       <axis xyz="1 0 0"/>
       <parent link="cell_element1_base"/>
       <child link="cell_element2_base"/>
    </joint>
- <xacro:property name="this_robot_name" value="cell_element1_" />
+  <xacro:property name="this_robot_name" value="cell_element1_" />
   <xacro:include filename="$(find robotic_cell_description)/urdf/robot_arm.xacro" >
   </xacro:include>
-   <xacro:property name="this_robot_name" value="cell_element2_" />
+  <xacro:property name="this_robot_name" value="cell_element2_" />
   <xacro:include filename="$(find robotic_cell_description)/urdf/robot_arm.xacro" >
   </xacro:include>

Commit message: experimet: recursive join urdfs from yaml dfn

File: urdf/robotic_cell.urdf.xacro (robot description, xacro)
@@ -1,19 +1,32 @@
 <?xml version="1.0"?>
 <robot xmlns:xacro="http://www.ros.org/wiki/xacro"  name="robotic_cell">
+  <xacro:macro name="loop_code" params="current_i names_vector yaml_data_dictionary"  >
+    <xacro:property name="current_name" value="${names_vector[current_i]}"/>
+    <xacro:property name="current_package_name" value="${yaml_data_dictionary[current_name]['package_name']}" />
+    <xacro:property name="current_urdf_name" value="${yaml_data_dictionary[current_name]['urdf_name']}" />
+    <xacro:property name="this_robot_name" value="${current_name + '_'}" />
+    <joint name="${this_robot_name + 'module_pose'}" type="fixed">
+        <origin xyz="${yaml_data_dictionary[current_name]['x']} ${yaml_data_dictionary[current_name]['y']} ${yaml_data_dictionary[current_name]['z']}" rpy="${yaml_data_dictionary[current_name]['er']} ${yaml_data_dictionary[current_name]['ep']} ${yaml_data_dictionary[current_name]['ey']}" />
+        <axis xyz="1 0 0"/>
+        <parent link="${yaml_data_dictionary[current_name]['parrent']}"/>
+        <child link="${this_robot_name + 'base'}"/>
+    </joint>
+    <xacro:include filename="$(find  ${current_package_name})/urdf/${current_urdf_name}" >
+    </xacro:include>
+  </xacro:macro>
+  <xacro:macro name="loop" params="current_i names_vector yaml_data_dictionary">
+      <!-- call some macros or do other things -->
+      <xacro:if value="${current_i}">
+          <xacro:loop_code current_i="${current_i-1}"  names_vector = "${list_of_active_elements_names}" yaml_data_dictionary="${yaml_data_dictionary}" />
+          <xacro:loop current_i="${current_i-1}"  names_vector = "${list_of_active_elements_names}" yaml_data_dictionary="${yaml_data_dictionary}"/>
+      </xacro:if>
+  </xacro:macro>
   <xacro:property name="yaml_file" value="$(find robotic_cell_description)/config/active_config.yaml" />
-  <xacro:property name="active_config" value="${load_yaml(yaml_file)}"/>
+  <xacro:property name="active_config" value="${xacro.load_yaml(yaml_file)}"/>
   <xacro:property name="current_connection_name" value="first_connection"/>
   <xacro:property name="connection_config" value="${active_config[current_connection_name]}"/>
-  <joint name="togehter" type="fixed">
-      <origin xyz="${connection_config['x']} ${connection_config['y']} ${connection_config['z']}" rpy="0 0 0"/>
-      <axis xyz="1 0 0"/>
-      <parent link="cell_element1_base"/>
-      <child link="cell_element2_base"/>
-   </joint>
-  <xacro:property name="this_robot_name" value="cell_element1_" />
-  <xacro:include filename="$(find robotic_cell_description)/urdf/robot_arm.xacro" >
-  </xacro:include>
-  <xacro:property name="this_robot_name" value="cell_element2_" />
-  <xacro:include filename="$(find robotic_cell_description)/urdf/robot_arm.xacro" >
-  </xacro:include>
+  <xacro:property name="list_of_active_elements_names" value="${active_config['active_description_elements']}"/>
+  <link name="robotic_cell_base">
+  </link>
+  <xacro:loop current_i="${len(list_of_active_elements_names)}" names_vector = "${list_of_active_elements_names}" yaml_data_dictionary="${active_config}"/>
 </robot>
